Commit message: Imagen de referencia

File: urdf/LeggedRobot.urdf (robot description, URDF)
Before this commit: robot cuadrupedo, 13 links, 12 joints
Links:
- link Bl_link_3: geometry visual box size=0.1 0.07 0.14
- link Br_link_3: geometry visual box size=0.1 0.07 0.14
- link Fl_link_3: geometry visual box size=0.1 0.07 0.14
- link Fr_link_3: geometry visual box size=0.1 0.07 0.14
